File: Assets/PCB Files/UGV.kicad_pcb (KiCad board)
At the start: 2 copper layers, 122 x 156.5 mm, 77 parts, among them J13 USB3_A, J15 Screw_Terminal_01x12, J16 Screw_Terminal_01x12, J17 Screw_Terminal_01x12, J18 Screw_Terminal_01x12, U1 INA219AxDCN, U2 LMR33630ADDA, U3 SN74LVC8T245, U4 Teensy4.1, U5 SN74LVC8T245

Commit message: PCB Done
Parts:
- removed U1: INA219AxDCN, Package_TO_SOT_SMD:SOT-23-8
- added Q1: AO3400A, Package_TO_SOT_SMD:SOT-23, F.Cu at (74.1, 131.0)
- added R3: 10k, Resistor_SMD:R_0402_1005Metric, F.Cu at (70.9, 130.0)
- R2: value 0.01 -> 100
- U2: footprint LMR33630AQRNXTQ1:CONV_LMR33620BRNXT -> LMR33630ADDA:VREG_LM5017MR_NOPB
- moved R2 104.9 mm to (72.7, 128.1)
- moved G*** 91.5 mm to (95.5, 23.0)
- moved C5 44.1 mm to (113.5, 71.0), turned to -90 degrees
- moved C8 41.5 mm to (103.0, 113.6), turned to 90 degrees
- moved C9 41.5 mm to (103.0, 118.6)
- moved Flysky1 41.4 mm to (99.1, 126.1)
- moved Flysky2 41.4 mm to (86.1, 126.1)
- moved U5 41.4 mm to (92.8, 115.9)
- moved Enc1 40.7 mm to (111.2, 57.5)
- moved Enc2 40.7 mm to (111.2, 50.5)
- moved Enc3 40.7 mm to (99.2, 50.5)
- moved Enc4 40.7 mm to (99.2, 57.5)
- moved J15 39.1 mm to (112.0, 105.5)
- moved J16 39.1 mm to (80.0, 105.5)
- moved J17 39.1 mm to (112.1, 79.0)
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Connections:
- C12 pad 1: Net-(U1-IN-) -> Net-(C12-Pad1)
- C3 pad 2: Net-(C3-Pad2) -> /Vin
- C5 pad 2: Net-(U3-V_{CCA}) -> /3V3
- C8 pad 2: Net-(U5-V_{CCA}) -> /3V3
- C9 pad 2: Net-(C9-Pad2) -> /Vout
- Cp3 pad 1: Net-(U1-IN-) -> Net-(C12-Pad1)
- Enc1 pad 1: unconnected-(Enc1-Pad1) -> Net-(U3-A1)
- Enc1 pad 2: unconnected-(Enc1-Pad2) -> Net-(U3-A2)
- Enc2 pad 1: unconnected-(Enc2-Pad1) -> Net-(U3-A3)
- Enc2 pad 2: unconnected-(Enc2-Pad2) -> Net-(U3-A4)
- Enc3 pad 1: unconnected-(Enc3-Pad1) -> Net-(U3-A5)
- Enc3 pad 2: unconnected-(Enc3-Pad2) -> Net-(U3-A6)
- Enc4 pad 1: unconnected-(Enc4-Pad1) -> Net-(U3-A7)
- Enc4 pad 2: unconnected-(Enc4-Pad2) -> Net-(U3-A8)
- FB1 pad 1: Net-(U1-IN-) -> Net-(C12-Pad1)
- Flysky1 pad 1: unconnected-(Flysky1-Pad1) -> Net-(U5-B1)
- Flysky1 pad 2: unconnected-(Flysky1-Pad2) -> Net-(U5-B2)
- Flysky1 pad 3: unconnected-(Flysky1-Pad3) -> Net-(U5-B3)
- Flysky1 pad 4: unconnected-(Flysky1-Pad4) -> Net-(U5-B4)
- Flysky2 pad 1: unconnected-(Flysky2-Pad1) -> Net-(U5-B5)
- Flysky2 pad 2: unconnected-(Flysky2-Pad2) -> Net-(U5-B6)
- Flysky2 pad 3: unconnected-(Flysky2-Pad3) -> Net-(U5-B7)
- Flysky2 pad 4: unconnected-(Flysky2-Pad4) -> Net-(U5-B8)
- J15 pad 1: unconnected-(J15-Pin_1-Pad1) -> /Vin
- J15 pad 10: unconnected-(J15-Pin_10-Pad10) -> /17
- J15 pad 11: unconnected-(J15-Pin_11-Pad11) -> /16
- J15 pad 12: unconnected-(J15-Pin_12-Pad12) -> /15
- J15 pad 2: unconnected-(J15-Pin_2-Pad2) -> GND
- J15 pad 3: unconnected-(J15-Pin_3-Pad3) -> /3V3
- J15 pad 4: unconnected-(J15-Pin_4-Pad4) -> /23
- J15 pad 5: unconnected-(J15-Pin_5-Pad5) -> /22
- J15 pad 6: unconnected-(J15-Pin_6-Pad6) -> /21
- J15 pad 7: unconnected-(J15-Pin_7-Pad7) -> /20
- J15 pad 8: unconnected-(J15-Pin_8-Pad8) -> /19
- J15 pad 9: unconnected-(J15-Pin_9-Pad9) -> /18
- J16 pad 1: unconnected-(J16-Pin_1-Pad1) -> /14
- J16 pad 10: unconnected-(J16-Pin_10-Pad10) -> /35
- J16 pad 11: unconnected-(J16-Pin_11-Pad11) -> /34
- J16 pad 12: unconnected-(J16-Pin_12-Pad12) -> /33
- J16 pad 2: unconnected-(J16-Pin_2-Pad2) -> /13
- J16 pad 3: unconnected-(J16-Pin_3-Pad3) -> GND
- J16 pad 4: unconnected-(J16-Pin_4-Pad4) -> /41
- J16 pad 5: unconnected-(J16-Pin_5-Pad5) -> /40
- J16 pad 6: unconnected-(J16-Pin_6-Pad6) -> /39
- J16 pad 7: unconnected-(J16-Pin_7-Pad7) -> /38
- J16 pad 8: unconnected-(J16-Pin_8-Pad8) -> /37
- J16 pad 9: unconnected-(J16-Pin_9-Pad9) -> /36
- J17 pad 1: unconnected-(J17-Pin_1-Pad1) -> GND
- J17 pad 10: unconnected-(J17-Pin_10-Pad10) -> /8
- J17 pad 11: unconnected-(J17-Pin_11-Pad11) -> /9
- J17 pad 12: unconnected-(J17-Pin_12-Pad12) -> /10
- J17 pad 2: unconnected-(J17-Pin_2-Pad2) -> /0
- J17 pad 3: unconnected-(J17-Pin_3-Pad3) -> /1
- J17 pad 4: unconnected-(J17-Pin_4-Pad4) -> /2
- J17 pad 5: unconnected-(J17-Pin_5-Pad5) -> /3
- J17 pad 6: unconnected-(J17-Pin_6-Pad6) -> /4
- J17 pad 7: unconnected-(J17-Pin_7-Pad7) -> /5
- J17 pad 8: unconnected-(J17-Pin_8-Pad8) -> /6
- J17 pad 9: unconnected-(J17-Pin_9-Pad9) -> /7
- J18 pad 1: unconnected-(J18-Pin_1-Pad1) -> /11
- J18 pad 10: unconnected-(J18-Pin_10-Pad10) -> /30
- J18 pad 11: unconnected-(J18-Pin_11-Pad11) -> /31
- J18 pad 12: unconnected-(J18-Pin_12-Pad12) -> /32
- J18 pad 2: unconnected-(J18-Pin_2-Pad2) -> /12
- J18 pad 3: unconnected-(J18-Pin_3-Pad3) -> /3V3
- J18 pad 4: unconnected-(J18-Pin_4-Pad4) -> /24
- J18 pad 5: unconnected-(J18-Pin_5-Pad5) -> /25
- J18 pad 6: unconnected-(J18-Pin_6-Pad6) -> /26
- J18 pad 7: unconnected-(J18-Pin_7-Pad7) -> /27
- J18 pad 8: unconnected-(J18-Pin_8-Pad8) -> /28
- J18 pad 9: unconnected-(J18-Pin_9-Pad9) -> /29
- L1 pad 2: Net-(U1-IN+) -> Net-(C12-Pad1)
- LED1 pad 2: GND -> Net-(Q1-D)
- MD_DIR1 pad 1: unconnected-(MD_DIR1-Pad1) -> /12
- MD_DIR1 pad 2: unconnected-(MD_DIR1-Pad2) -> /11
- MD_DIR2 pad 1: unconnected-(MD_DIR2-Pad1) -> /26
- MD_DIR2 pad 2: unconnected-(MD_DIR2-Pad2) -> /27
- MD_PWM1 pad 1: unconnected-(MD_PWM1-Pad1) -> /9
- MD_PWM1 pad 2: unconnected-(MD_PWM1-Pad2) -> /10
- MD_PWM2 pad 1: unconnected-(MD_PWM2-Pad1) -> /29
- MD_PWM2 pad 2: unconnected-(MD_PWM2-Pad2) -> /28
- R2 pad 1: Net-(U1-IN+) -> Net-(Q1-G)
- R2 pad 2: Net-(U1-IN-) -> /41
- U3 pad 1: Net-(U3-V_{CCA}) -> /Vin
- U3 pad 10: unconnected-(U3-A8-Pad10) -> Net-(U3-A8)
- U3 pad 14: unconnected-(U3-B8-Pad14) -> /8
- U3 pad 15: unconnected-(U3-B7-Pad15) -> /7
- U3 pad 16: unconnected-(U3-B6-Pad16) -> /6
- U3 pad 17: unconnected-(U3-B5-Pad17) -> /5
- U3 pad 18: unconnected-(U3-B4-Pad18) -> /4
- U3 pad 19: unconnected-(U3-B3-Pad19) -> /3
- U3 pad 2: GND -> /Vin
- U3 pad 20: unconnected-(U3-B2-Pad20) -> /2
- U3 pad 21: unconnected-(U3-B1-Pad21) -> /1
- U3 pad 23: Net-(C3-Pad2) -> /3V3
- U3 pad 24: Net-(C3-Pad2) -> /3V3
- U3 pad 3: unconnected-(U3-A1-Pad3) -> Net-(U3-A1)
- U3 pad 4: unconnected-(U3-A2-Pad4) -> Net-(U3-A2)
- U3 pad 5: unconnected-(U3-A3-Pad5) -> Net-(U3-A3)
- U3 pad 6: unconnected-(U3-A4-Pad6) -> Net-(U3-A4)
- U3 pad 7: unconnected-(U3-A5-Pad7) -> Net-(U3-A5)
- U3 pad 8: unconnected-(U3-A6-Pad8) -> Net-(U3-A6)
- U3 pad 9: unconnected-(U3-A7-Pad9) -> Net-(U3-A7)
- U4 pad 1: unconnected-(U4-GND-Pad1) -> GND
- U4 pad 10: unconnected-(U4-8_TX2_IN1-Pad10) -> /8
- U4 pad 11: unconnected-(U4-9_OUT1C-Pad11) -> /9
- U4 pad 12: unconnected-(U4-10_CS_MQSR-Pad12) -> /10
- U4 pad 13: unconnected-(U4-11_MOSI_CTX1-Pad13) -> /11
- U4 pad 14: unconnected-(U4-12_MISO_MQSL-Pad14) -> /12
- U4 pad 15: unconnected-(U4-3V3-Pad15) -> /3V3
- U4 pad 16: unconnected-(U4-24_A10_TX6_SCL2-Pad16) -> /24
- U4 pad 17: unconnected-(U4-25_A11_RX6_SDA2-Pad17) -> /25
- U4 pad 18: unconnected-(U4-26_A12_MOSI1-Pad18) -> /26
- U4 pad 19: unconnected-(U4-27_A13_SCK1-Pad19) -> /27
- U4 pad 2: unconnected-(U4-0_RX1_CRX2_CS1-Pad2) -> /0
- U4 pad 20: unconnected-(U4-28_RX7-Pad20) -> /28
- U4 pad 21: unconnected-(U4-29_TX7-Pad21) -> /29
- U4 pad 22: unconnected-(U4-30_CRX3-Pad22) -> /30
- U4 pad 23: unconnected-(U4-31_CTX3-Pad23) -> /31
- U4 pad 24: unconnected-(U4-32_OUT1B-Pad24) -> /32
- U4 pad 25: unconnected-(U4-33_MCLK2-Pad25) -> /33
- U4 pad 26: unconnected-(U4-34_RX8-Pad26) -> /34
- U4 pad 27: unconnected-(U4-35_TX8-Pad27) -> /35
- U4 pad 28: unconnected-(U4-36_CS-Pad28) -> /36
- U4 pad 29: unconnected-(U4-37_CS-Pad29) -> /37
- U4 pad 3: unconnected-(U4-1_TX1_CTX2_MISO1-Pad3) -> /1
- U4 pad 30: unconnected-(U4-38_CS1_IN1-Pad30) -> /38
- U4 pad 31: unconnected-(U4-39_MISO1_OUT1A-Pad31) -> /39
- U4 pad 32: unconnected-(U4-40_A16-Pad32) -> /40
- U4 pad 33: unconnected-(U4-41_A17-Pad33) -> /41
- U4 pad 34: unconnected-(U4-GND-Pad34) -> GND
- U4 pad 35: unconnected-(U4-13_SCK_LED-Pad35) -> /13
- U4 pad 36: unconnected-(U4-14_A0_TX3_SPDIF_OUT-Pad36) -> /14
- U4 pad 37: unconnected-(U4-15_A1_RX3_SPDIF_IN-Pad37) -> /15
- U4 pad 38: unconnected-(U4-16_A2_RX4_SCL1-Pad38) -> /16
- U4 pad 39: unconnected-(U4-17_A3_TX4_SDA1-Pad39) -> /17
- U4 pad 4: unconnected-(U4-2_OUT2-Pad4) -> /2
- U4 pad 40: unconnected-(U4-18_A4_SDA-Pad40) -> /18
- U4 pad 41: unconnected-(U4-19_A5_SCL-Pad41) -> /19
- U4 pad 42: unconnected-(U4-20_A6_TX5_LRCLK1-Pad42) -> /20
- U4 pad 43: unconnected-(U4-21_A7_RX5_BCLK1-Pad43) -> /21
- U4 pad 44: unconnected-(U4-22_A8_CTX1-Pad44) -> /22
- U4 pad 45: unconnected-(U4-23_A9_CRX1_MCLK1-Pad45) -> /23
- U4 pad 46: unconnected-(U4-3V3-Pad46) -> /3V3
- U4 pad 47: unconnected-(U4-GND-Pad47) -> GND
- U4 pad 5: unconnected-(U4-3_LRCLK2-Pad5) -> /3
- U4 pad 6: unconnected-(U4-4_BCLK2-Pad6) -> /4
- U4 pad 7: unconnected-(U4-5_IN2-Pad7) -> /5
- U4 pad 8: unconnected-(U4-6_OUT1D-Pad8) -> /6
- U4 pad 9: unconnected-(U4-7_RX2_OUT1A-Pad9) -> /7
- U5 pad 1: Net-(U5-V_{CCA}) -> /3V3
- U5 pad 10: unconnected-(U5-A8-Pad10) -> /14
- U5 pad 14: unconnected-(U5-B8-Pad14) -> Net-(U5-B8)
- U5 pad 15: unconnected-(U5-B7-Pad15) -> Net-(U5-B7)
- U5 pad 16: unconnected-(U5-B6-Pad16) -> Net-(U5-B6)
- U5 pad 17: unconnected-(U5-B5-Pad17) -> Net-(U5-B5)
- U5 pad 18: unconnected-(U5-B4-Pad18) -> Net-(U5-B4)
- U5 pad 19: unconnected-(U5-B3-Pad19) -> Net-(U5-B3)
- U5 pad 20: unconnected-(U5-B2-Pad20) -> Net-(U5-B2)
- U5 pad 21: unconnected-(U5-B1-Pad21) -> Net-(U5-B1)
- U5 pad 23: Net-(C9-Pad2) -> /Vout
- U5 pad 24: Net-(C9-Pad2) -> /Vout
- U5 pad 3: unconnected-(U5-A1-Pad3) -> /23
- U5 pad 4: unconnected-(U5-A2-Pad4) -> /22
- U5 pad 5: unconnected-(U5-A3-Pad5) -> /21
- U5 pad 6: unconnected-(U5-A4-Pad6) -> /20
- U5 pad 7: unconnected-(U5-A5-Pad7) -> /19
- U5 pad 8: unconnected-(U5-A6-Pad8) -> /18
- U5 pad 9: unconnected-(U5-A7-Pad9) -> /15
Routing:
- net GND: track 0.00 -> 349.1 mm, vias 0 -> 199
- net /Vout: track 0.00 -> 206.6 mm
- net Net-(D1-A): track 0.00 -> 152.7 mm
- net /3V3: track 0.00 -> 59.6 mm
- net /Vin: track 0.00 -> 56.0 mm
- net Net-(Q1-D): track 0.00 -> 41.9 mm
- net Net-(12Vout1-PadP): track 0.00 -> 39.0 mm
- net /41: track 0.00 -> 28.2 mm
- net /11: track 0.00 -> 27.1 mm
- net /27: track 0.00 -> 26.2 mm
- net /12: track 0.00 -> 26.0 mm
- net /26: track 0.00 -> 25.1 mm
- net /14: track 0.00 -> 17.3 mm
- net /8: track 0.00 -> 17.3 mm
- net /29: track 0.00 -> 17.2 mm
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- added copper zone on F.Cu, net /Vout
- added copper zone on B.Cu, net GND
- added copper zone on F.Cu, net Net-(12Vout(C)1-PadP)
- added copper zone on F.Cu, net Net-(12Vout1-PadP)
- added copper zone on F.Cu, net Net-(C12-Pad1)
- added copper zone on F.Cu, net Net-(D1-A)
- added copper zone on F.Cu, net Net-(U2-SW)
Other:
- board size 122 x 156.5 mm -> 120.6 x 156.5 mm
