File: Assets/PCB Files/UGV.kicad_pcb (KiCad board)
At the start: 2 copper layers, 120.6 x 156.5 mm, 78 parts, among them J13 USB3_A, J15 Screw_Terminal_01x12, J16 Screw_Terminal_01x12, J17 Screw_Terminal_01x12, J18 Screw_Terminal_01x12, Q1 AO3400A, U2 LMR33630ADDA, U3 SN74LVC8T245, U4 Teensy4.1, U5 SN74LVC8T245

Commit message: Completed Routing of the PCB
Parts:
- added 5V_ScrewTerm1: Screw_Terminal_01x02, TerminalBlock_Phoenix:TerminalBlock_Phoenix_MKDS-1,5-2-5.08_1x02_P5.08mm_Horizontal, F.Cu at (115.7, 154.0)
- added D2: LED, LED_SMD:LED_1206_3216Metric_Pad1.42x1.75mm_HandSolder, F.Cu at (56.1, 22.6)
- added D3: LED, LED_SMD:LED_1206_3216Metric_Pad1.42x1.75mm_HandSolder, F.Cu at (34.3, 83.8)
- added D4: LED, LED_SMD:LED_1206_3216Metric_Pad1.42x1.75mm_HandSolder, F.Cu at (20.9, 46.9)
- added D5: LED, LED_SMD:LED_1206_3216Metric_Pad1.42x1.75mm_HandSolder, F.Cu at (37.5, 132.2)
- added D6: LED, LED_SMD:LED_1206_3216Metric_Pad1.42x1.75mm_HandSolder, F.Cu at (117.3, 106.4)
- added LED2: Screw_Terminal_01x02, TerminalBlock_Phoenix:TerminalBlock_Phoenix_MKDS-1,5-2-5.08_1x02_P5.08mm_Horizontal, F.Cu at (41.9, 62.2)
- added Q2: AO3400A, Package_TO_SOT_SMD:SOT-23_Handsoldering, F.Cu at (74.3, 117.9)
- added Q3: AO3400A, Package_TO_SOT_SMD:SOT-23_Handsoldering, F.Cu at (43.6, 72.0)
- added R10: 4.7 kohm, Resistor_SMD:R_1206_3216Metric_Pad1.30x1.75mm_HandSolder, F.Cu at (39.6, 83.8)
- added R11: 390 ohm, Resistor_SMD:R_1206_3216Metric_Pad1.30x1.75mm_HandSolder, F.Cu at (32.0, 132.2)
- added R12: 390 ohm, Resistor_SMD:R_1206_3216Metric_Pad1.30x1.75mm_HandSolder, F.Cu at (117.3, 111.7)
- added R4: 100, Resistor_SMD:R_0805_2012Metric_Pad1.20x1.40mm_HandSolder, F.Cu at (77.6, 114.9)
- added R5: 100k, Resistor_SMD:R_1206_3216Metric_Pad1.30x1.75mm_HandSolder, F.Cu at (73.6, 113.0)
- added R6: 100, Resistor_SMD:R_0805_2012Metric_Pad1.20x1.40mm_HandSolder, F.Cu at (46.6, 75.1)
- added R7: 100k, Resistor_SMD:R_1206_3216Metric_Pad1.30x1.75mm_HandSolder, F.Cu at (48.3, 71.1)
- added R8: 1.8 kohm, Resistor_SMD:R_1206_3216Metric_Pad1.30x1.75mm_HandSolder, F.Cu at (56.1, 28.0)
- added R9: 1.8 kohm, Resistor_SMD:R_1206_3216Metric_Pad1.30x1.75mm_HandSolder, F.Cu at (20.9, 52.2)
- Cout1: footprint Capacitor_SMD:C_0603_1608Metric_Pad1.08x0.95mm_HandSolder -> Capacitor_SMD:C_1210_3225Metric_Pad1.33x2.70mm_HandSolder
- Q1: footprint Package_TO_SOT_SMD:SOT-23 -> Package_TO_SOT_SMD:SOT-23_Handsoldering
- moved Laser1 9.56 mm to (115.3, 142.2), turned to 90 degrees
- moved Cvcc1 9.12 mm to (43.0, 121.9), turned to -45 degrees
- moved Cout2 9.04 mm to (42.4, 129.4), turned to -90 degrees
- moved Cff1 8.37 mm to (36.6, 126.8)
- moved Rfbt1 8.26 mm to (39.3, 126.3)
- moved R2 6.66 mm to (67.6, 123.8)
- moved Cout1 6.37 mm to (46.0, 129.5), turned to -90 degrees
- moved R3 6.19 mm to (64.9, 128.6), turned to 90 degrees
- moved Rfbb1 5.82 mm to (35.1, 123.4)
- moved Q1 5.69 mm to (69.3, 127.8)
- moved LED1 5.67 mm to (107.3, 142.2)
- moved Flysky1 4.95 mm to (103.7, 127.9), turned to 180 degrees
- moved L2 4.87 mm to (54.6, 122.7)
- moved Flysky2 3.25 mm to (88.8, 127.9), turned to 180 degrees
- moved 12Vout(C)1 2.29 mm to (65.9, 6.52)
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Connections:
- Laser1 pad 2: GND -> Net-(Q2-D)
- PWRin1 pad 1: (no net) -> GND
- PWRin1 pad 2: (no net) -> Net-(D1-A)
- U4 pad 49: unconnected-(U4-VUSB-Pad49) -> (no net)
- U4 pad 50: unconnected-(U4-VBAT-Pad50) -> (no net)
- U4 pad 51: unconnected-(U4-3V3-Pad51) -> (no net)
- U4 pad 52: unconnected-(U4-GND-Pad52) -> (no net)
- U4 pad 53: unconnected-(U4-PROGRAM-Pad53) -> (no net)
- U4 pad 54: unconnected-(U4-ON_OFF-Pad54) -> (no net)
- U4 pad 55: unconnected-(U4-5V-Pad55) -> (no net)
- U4 pad 56: unconnected-(U4-D--Pad56) -> (no net)
- U4 pad 57: unconnected-(U4-D+-Pad57) -> (no net)
- U4 pad 58: unconnected-(U4-GND-Pad58) -> (no net)
- U4 pad 59: unconnected-(U4-GND-Pad59) -> (no net)
- U4 pad 60: unconnected-(U4-R+-Pad60) -> (no net)
- U4 pad 61: unconnected-(U4-LED-Pad61) -> (no net)
- U4 pad 62: unconnected-(U4-T--Pad62) -> (no net)
- U4 pad 63: unconnected-(U4-T+-Pad63) -> (no net)
- U4 pad 64: unconnected-(U4-GND-Pad64) -> (no net)
- U4 pad 65: unconnected-(U4-R--Pad65) -> (no net)
- U4 pad 66: unconnected-(U4-D--Pad66) -> (no net)
- U4 pad 67: unconnected-(U4-D+-Pad67) -> (no net)
Routing:
- net Net-(Q2-D): track 0.00 -> 54.9 mm
- net Net-(D4-A): track 39.0 -> 69.6 mm
- net /Vout: track 206.6 -> 230.4 mm
- net Net-(U2-FB): track 4.61 -> 15.9 mm
- net Net-(D1-A): track 154.5 -> 164.5 mm
- net /M1: track 0.00 -> 9.73 mm
- net /13: track 5.97 -> 13.2 mm
- net /32: track 6.04 -> 12.3 mm
- net Net-(Q2-G): track 0.00 -> 5.12 mm
- net Net-(Q3-G): track 0.00 -> 5.12 mm
- net /Vin: track 56.0 -> 60.5 mm
- net GND: track 349.1 -> 352.4 mm, vias 199 -> 213
- net /41: track 28.2 -> 25.4 mm
- net Net-(D3-K): track 0.00 -> 2.29 mm
- net Net-(D5-K): track 0.00 -> 2.29 mm
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Other:
- board text removed: "PWRin1"
