File: Assets/PCB Files/UGV.kicad_sch (KiCad schematic)
At the start: 76 parts, among them J13 USB3_A, J15 Screw_Terminal_01x12, J16 Screw_Terminal_01x12, J17 Screw_Terminal_01x12, J18 Screw_Terminal_01x12, U1 INA219AxDCN, U2 LMR33630ADDA, U3 SN74LVC8T245, U4 Teensy4.1, U5 SN74LVC8T245

Commit message: PCB Done
Parts:
- removed U1: INA219AxDCN, Package_TO_SOT_SMD:SOT-23-8, symbol Sensor_Energy:INA219AxDCN
- added Q1: AO3400A, Package_TO_SOT_SMD:SOT-23, symbol Transistor_FET:AO3400A
- added R3: 10k, Resistor_SMD:R_0402_1005Metric, symbol Device:R
- R2: value 0.01 -> 100
- U2: footprint LMR33630AQRNXTQ1:CONV_LMR33620BRNXT -> LMR33630ADDA:VREG_LM5017MR_NOPB
Connections:
- net GND: now also J15.2 (Pin_2), J16.3 (Pin_3), J17.1 (Pin_1), U4.1 (GND), U4.34 (GND), U4.47 (GND), Q1.2 (S), R3.1; no longer LED1.2, U3.2 (DIR)
- net Vin: now also C3.2, J15.1 (Pin_1), U3.1 (V_{CCA}), U3.2 (DIR)
- net Vout: now also C9.2, U5.23 (V_{CCB}), U5.24 (V_{CCB})
- net at L1.2: now also C12.1, Cp3.1, FB1.1; no longer R2.1
- net 3V3: now reaches C8.2, U5.1 (V_{CCA})
- net 3V3: now also C5.2, J15.3 (Pin_3), J18.3 (Pin_3), U3.23 (V_{CCB}), U3.24 (V_{CCB}), U4.15 (3V3), U4.46 (3V3)
- net 14: now reaches U5.10 (A8)
- net 14: now also J16.1 (Pin_1), U4.36 (14_A0_TX3_SPDIF_OUT)
- net at U5.14 (B8): now also Flysky2.4
- net at U5.15 (B7): now also Flysky2.3
- net at U5.16 (B6): now also Flysky2.2
- net at U5.17 (B5): now also Flysky2.1
- net at U5.18 (B4): now also Flysky1.4
- net at U5.19 (B3): now also Flysky1.3
- net at U5.20 (B2): now also Flysky1.2
- net at U5.21 (B1): now also Flysky1.1
- net 23: now reaches U5.3 (A1)
- net 23: now also J15.4 (Pin_4), U4.45 (23_A9_CRX1_MCLK1)
- net 22: now reaches U5.4 (A2)
- net 22: now also J15.5 (Pin_5), U4.44 (22_A8_CTX1)
- net 21: now reaches U5.5 (A3)
- net 21: now also J15.6 (Pin_6), U4.43 (21_A7_RX5_BCLK1)
- net 20: now reaches U5.6 (A4)
- net 20: now also J15.7 (Pin_7), U4.42 (20_A6_TX5_LRCLK1)
- net 19: now reaches U5.7 (A5)
- net 19: now also J15.8 (Pin_8), U4.41 (19_A5_SCL)
- net 18: now reaches U5.8 (A6)
- net 18: now also J15.9 (Pin_9), U4.40 (18_A4_SDA)
- net 15: now reaches U5.9 (A7)
- net 15: now also J15.12 (Pin_12), U4.37 (15_A1_RX3_SPDIF_IN)
- net at U3.10 (A8): now also Enc4.2
- net 8: now reaches U3.14 (B8)
- net 8: now also J17.10 (Pin_10), U4.10 (8_TX2_IN1)
- net 7: now reaches U3.15 (B7)
- net 7: now also J17.9 (Pin_9), U4.9 (7_RX2_OUT1A)
- net 6: now reaches U3.16 (B6)
- net 6: now also J17.8 (Pin_8), U4.8 (6_OUT1D)
- net 5: now reaches U3.17 (B5)
- net 5: now also J17.7 (Pin_7), U4.7 (5_IN2)
- net 4: now reaches U3.18 (B4)
- net 4: now also J17.6 (Pin_6), U4.6 (4_BCLK2)
- net 3: now reaches U3.19 (B3)
- net 3: now also J17.5 (Pin_5), U4.5 (3_LRCLK2)
- net 2: now reaches U3.20 (B2)
- net 2: now also J17.4 (Pin_4), U4.4 (2_OUT2)
- net 1: now reaches U3.21 (B1)
- net 1: now also J17.3 (Pin_3), U4.3 (1_TX1_CTX2_MISO1)
- net at U3.3 (A1): now also Enc1.1
- net at U3.4 (A2): now also Enc1.2
- net at U3.5 (A3): now also Enc2.1
- net at U3.6 (A4): now also Enc2.2
- net at U3.7 (A5): now also Enc3.1
- net at U3.8 (A6): now also Enc3.2
- net at U3.9 (A7): now also Enc4.1
- net 11: now reaches J18.1 (Pin_1)
- net 11: now also MD_DIR1.2, U4.13 (11_MOSI_CTX1)
- net 30: now reaches J18.10 (Pin_10)
- net 30: now also U4.22 (30_CRX3)
- net 31: now reaches J18.11 (Pin_11)
- net 31: now also U4.23 (31_CTX3)
- net 32: now reaches J18.12 (Pin_12)
- net 32: now also U4.24 (32_OUT1B)
- net 12: now reaches J18.2 (Pin_2)
- net 12: now also MD_DIR1.1, U4.14 (12_MISO_MQSL)
- net 24: now reaches J18.4 (Pin_4)
- net 24: now also U4.16 (24_A10_TX6_SCL2)
- net 25: now reaches J18.5 (Pin_5)
- net 25: now also U4.17 (25_A11_RX6_SDA2)
- net 26: now reaches J18.6 (Pin_6)
- net 26: now also MD_DIR2.1, U4.18 (26_A12_MOSI1)
- net 27: now reaches J18.7 (Pin_7)
- net 27: now also MD_DIR2.2, U4.19 (27_A13_SCK1)
- net 28: now reaches J18.8 (Pin_8)
- net 28: now also MD_PWM2.2, U4.20 (28_RX7)
- net 29: now reaches J18.9 (Pin_9)
- net 29: now also MD_PWM2.1, U4.21 (29_TX7)
- net 17: now reaches J15.10 (Pin_10)
- net 17: now also U4.39 (17_A3_TX4_SDA1)
- net 16: now reaches J15.11 (Pin_11)
- net 16: now also U4.38 (16_A2_RX4_SCL1)
- net 9: now reaches MD_PWM1.1
- net 9: now also J17.11 (Pin_11), U4.11 (9_OUT1C)
- net 10: now reaches MD_PWM1.2
- net 10: now also J17.12 (Pin_12), U4.12 (10_CS_MQSR)
- net 35: now reaches J16.10 (Pin_10)
- net 35: now also U4.27 (35_TX8)
- net 34: now reaches J16.11 (Pin_11)
- net 34: now also U4.26 (34_RX8)
- net 33: now reaches J16.12 (Pin_12)
- net 33: now also U4.25 (33_MCLK2)
- net 13: now reaches J16.2 (Pin_2)
- net 13: now also U4.35 (13_SCK_LED)
- net 41: now reaches J16.4 (Pin_4)
- net 41: now also R2.2, U4.33 (41_A17)
- net 40: now reaches J16.5 (Pin_5)
- net 40: now also U4.32 (40_A16)
- net 39: now reaches J16.6 (Pin_6)
- net 39: now also U4.31 (39_MISO1_OUT1A)
- net 38: now reaches J16.7 (Pin_7)
- net 38: now also U4.30 (38_CS1_IN1)
- net 37: now reaches J16.8 (Pin_8)
- net 37: now also U4.29 (37_CS)
- net 36: now reaches J16.9 (Pin_9)
- net 36: now also U4.28 (36_CS)
- net 0: now reaches J17.2 (Pin_2)
- net 0: now also U4.2 (0_RX1_CRX2_CS1)
- new net: Q1.1 (G), R2.1, R3.2
- new net: LED1.2, Q1.3 (D)
- no-connect marks 26 -> 29
