File: Assets/PCB Files/.history/UGV.kicad_sch (KiCad schematic)
At the start: 77 parts, among them J13 USB3_A, J15 Screw_Terminal_01x12, J16 Screw_Terminal_01x12, J17 Screw_Terminal_01x12, J18 Screw_Terminal_01x12, Q1 AO3400A, U2 LMR33630ADDA, U3 SN74LVC8T245, U4 Teensy4.1, U5 SN74LVC8T245

Commit message: Completed Routing of the PCB
Parts:
- added 5V_ScrewTerm1, LED2: Screw_Terminal_01x02, TerminalBlock_Phoenix:TerminalBlock_Phoenix_MKDS-1,5-2-5.08_1x02_P5.08mm_Horizontal, symbol Connector:Screw_Terminal_01x02
- added D2, D3, D4, D5, D6: LED, LED_SMD:LED_1206_3216Metric_Pad1.42x1.75mm_HandSolder, symbol Device:LED
- added Q2, Q3: AO3400A, Package_TO_SOT_SMD:SOT-23_Handsoldering, symbol Transistor_FET:AO3400A
- added R10: 4.7 kohm, Resistor_SMD:R_1206_3216Metric_Pad1.30x1.75mm_HandSolder, symbol Device:R
- added R11, R12: 390 ohm, Resistor_SMD:R_1206_3216Metric_Pad1.30x1.75mm_HandSolder, symbol Device:R
- added R4, R6: 100, Resistor_SMD:R_0805_2012Metric_Pad1.20x1.40mm_HandSolder, symbol Device:R
- added R5, R7: 100k, Resistor_SMD:R_1206_3216Metric_Pad1.30x1.75mm_HandSolder, symbol Device:R
- added R8, R9: 1.8 kohm, Resistor_SMD:R_1206_3216Metric_Pad1.30x1.75mm_HandSolder, symbol Device:R
- Cout1: footprint Capacitor_SMD:C_0603_1608Metric_Pad1.08x0.95mm_HandSolder -> Capacitor_SMD:C_1210_3225Metric_Pad1.33x2.70mm_HandSolder
- Q1: footprint Package_TO_SOT_SMD:SOT-23 -> Package_TO_SOT_SMD:SOT-23_Handsoldering
Connections:
- net 13: now also R4.2
- net 32: now also R6.2
- net GND: now also PWRin1.1, 5V_ScrewTerm1.1 (Pin_1), Q2.2 (S), Q3.2 (S), R10.2, R11.2, R12.2, R5.1, R7.1, R8.2, R9.2; no longer Laser1.2, PWRin1.N
- net Vin: now also D6.2 (A)
- net Vout: now also 5V_ScrewTerm1.2 (Pin_2), D5.2 (A)
- net at 12Vout1.P, BUCKin1.P, C7.1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: now also D4.2 (A), LED2.2 (Pin_2)
- net at BUCKout1.P, Chf1.1, Cin1.1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: now also PWRin1.2, D3.2 (A); no longer PWRin1.P
- net at 12Vout(C)1.P, C15.1, C16.1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: now also D2.2 (A)
- new net: Q2.1 (G), R4.1, R5.2
- new net: D2.1 (K), R8.1
- new net: D6.1 (K), R12.1
- new net: D5.1 (K), R11.1
- new net: Q3.1 (G), R6.1, R7.2
- new net: D4.1 (K), R9.1
- new net: D3.1 (K), R10.1
- new net: Laser1.2, Q2.3 (D)
- new net M1: LED2.1 (Pin_1), Q3.3 (D)
Other:
- moved on the sheet: Q1, R2, R3, Servo1
